File: Eagle/PeakShaver.brd (EAGLE design)
At the start: 29.4 x 77.1 mm, 19 parts, among them J1 A5V, J2 SM5V, J3 RJ11, J4 RGB Button, T1 BC547, X4 RS485

Commit message: fixed bug in P1 connection
P1 ground and data line were swapped in version 0.9
Connections:
- net D: now also J3.5; no longer J3.3
- net GND: now also J3.3; no longer J3.5
Routing:
- net D: track 53.4 -> 61.2 mm
- net RTS: track 10.8 -> 13.8 mm
- net BASE: track 63.4 -> 66.0 mm, vias 1 -> 0
- net B: track 43.9 -> 46.1 mm
- net RX: track 38.4 -> 40.4 mm
- net DIR: track 9.04 -> 10.4 mm
- net DI: track 4.34 -> 5.57 mm
- net RO: track 5.39 -> 6.40 mm
- net +5V: track 104.3 -> 104.2 mm, vias 2 -> 0
Other:
- board text added: "PeakShaver 1.0"
- board text removed: "PeakShaver 0.9"
